Commit message: second commit

File: Collision_Avoidance/wrs_gazebo/mobile_dual_arm/urdf/mobile_dual_arm.xacro (robot description, xacro)
@@ -3,5 +3,5 @@
   <xacro:include filename="$(find single_arm_description)/urdf/single_arm.xacro" />
   <xacro:include filename="$(find Slide_rail)/urdf/Slide_rail.xacro" />
-  <xacro:include filename="$(find suction_urdf)/urdf/suction_urdf.xacro" />
+  <!-- <xacro:include filename="$(find suction_urdf)/urdf/suction_urdf.xacro" /> -->
   <!-- <xacro:include filename="$(find single_arm_description)/urdf/materials.xacro" /> -->
   <xacro:include filename="$(find mobile_dual_arm)/urdf/mobile_dual_arm.gazebo" />
@@ -82,4 +82,49 @@
     <child link="Base"/>
   </joint-->
+  <link
+    name="peg_link">
+    <inertial>
+      <origin
+        xyz="0 0 0"
+        rpy="0 0 0" />
+      <mass
+        value="0.5" />
+      <inertia
+        ixx="0.1"
+        ixy="0"
+        ixz="0"
+        iyy="0.1"
+        iyz="0"
+        izz="0.1" />
+    </inertial>
+    <visual>
+      <origin
+        xyz="0 0 0"
+        rpy="0 0 0" />
+      <geometry>
+        <cylinder length="0.06" radius="0.01"/>
+      </geometry>
+      <material
+        name="">
+        <color
+          rgba="0.1 0.1 0.1 1" />
+      </material>
+    </visual>
+    <collision>
+      <origin
+        xyz="0 0 0"
+        rpy="0 0 0" />
+      <geometry>
+        <cylinder length="0.06" radius="0.01"/>
+      </geometry>
+    </collision>
+  </link>
+  <joint name="fixed6" type="fixed">
+    <origin
+      xyz="-0.01785 0 0.05"
+      rpy="0 0 0" />
+    <parent link="r_left_inner_finger"/>
+    <child link="peg_link"/>
+  </joint>
   <joint name="fixed1" type="fixed">
     <origin

File: Collision_Avoidance/wrs_gazebo/robotiq_arg85_description/urdf/robotiq_arg85_description.urdf.xacro (robot description, xacro)
@@ -86,8 +86,8 @@
   <joint
     name="${side}_finger_joint"
-    type="revolute">
+    type="fixed">
     <origin
       xyz="0.0306011444260539 0 0.0627920162695395"
-      rpy="0 0 0" />
+      rpy="0 -0.55441176 0" />
     <parent
       link="${side}_robotiq_85_base_link" />
@@ -197,8 +197,8 @@
   <joint
     name="${side}_left_inner_knuckle_joint"
-    type="revolute">
+    type="fixed">
     <origin
       xyz="0.0127000000001501 0 0.0693074999999639"
-      rpy="0 0 0" />
+      rpy="0 -0.55441176 0" />
     <parent
       link="${side}_robotiq_85_base_link" />
@@ -255,8 +255,8 @@
   <joint
     name="${side}_left_inner_finger_joint"
-    type="revolute">
+    type="fixed">
     <origin
       xyz="0.034585310861294 0 0.0454970193817975"
-      rpy="0 0 0" />
+      rpy="0 0.55441176 0" />
     <parent
       link="${side}_left_inner_knuckle" />
@@ -313,8 +313,8 @@
   <joint
     name="${side}_right_inner_knuckle_joint"
-    type="revolute">
+    type="fixed">
     <origin
       xyz="-0.0126999999998499 0 0.0693075000000361"
-      rpy="0 0 3.14159265358979" />
+      rpy="0 -0.55441176 3.14159265358979" />
     <parent
       link="${side}_robotiq_85_base_link" />
@@ -371,8 +371,8 @@
   <joint
     name="${side}_right_inner_finger_joint"
-    type="revolute">
+    type="fixed">
     <origin
       xyz="0.0341060475457406 0 0.0458573878541688"
-      rpy="0 0 0" />
+      rpy="0 0.55441176 0" />
     <parent
       link="${side}_right_inner_knuckle" />
@@ -429,8 +429,8 @@
   <joint
     name="${side}_right_outer_knuckle_joint"
-    type="revolute">
+    type="fixed">
     <origin
       xyz="-0.0306011444258893 0 0.0627920162695395"
-      rpy="0 0 3.14159265358979" />
+      rpy="0 -0.55441176 3.14159265358979" />
     <parent
       link="${side}_robotiq_85_base_link" />
@@ -510,5 +510,5 @@
       xyz="0 1 0" />
   </joint>
-  <transmission name="${side}_tran1">
+  <!-- <transmission name="${side}_tran1">
     <type>transmission_interface/SimpleTransmission</type>
     <joint name="${side}_finger_joint">
@@ -569,5 +569,5 @@
       <mechanicalReduction>1</mechanicalReduction>
     </actuator>
-  </transmission>
+  </transmission> -->
   <xacro:robotiq_arg85_gazebo side="${side}"/>
   </xacro:macro>
